Commit message: updated

File: src/rover_robot/urdf/robot.urdf.xacro (robot description, xacro)
@@ -33,4 +33,64 @@
         </inertial>
     </link>
+    <joint name="camera_arm_joint" type="revolute">
+        <parent link="chassis"/>
+        <child link="camera_arm"/>
+        <origin xyz="0.15 0 0.05" rpy="0 0 0"/>
+        <axis xyz="0 1 0"/>
+        <limit lower="-0.785" upper="0.785" effort="10.0" velocity="1.0"/>
+    </joint>
+    <link name="camera_arm">
+        <visual>
+            <origin xyz="0 0 0.05" rpy="0 0 0"/>
+            <geometry>
+                <box size="0.04 0.04 0.1"/>
+            </geometry>
+            <material name="rover_body"/>
+        </visual>
+        <collision>
+            <origin xyz="0 0 0.05" rpy="0 0 0"/>
+            <geometry>
+                <box size="0.04 0.04 0.1"/>
+            </geometry>
+        </collision>
+        <inertial>
+            <origin xyz="0 0 0.05" rpy="0 0 0"/>
+            <mass value="0.1"/>
+            <inertia ixx="0.0001" ixy="0.0" ixz="0.0" iyy="0.0001" iyz="0.0" izz="0.0001"/>
+        </inertial>
+    </link>
+    <joint name="camera_joint" type="fixed">
+        <parent link="camera_arm"/>
+        <child link="camera_link"/>
+        <origin xyz="0.02 0 0.08" rpy="0 0 0"/>
+    </joint>
+    <link name="camera_link">
+        <visual>
+            <geometry><box size="0.02 0.04 0.04"/></geometry>
+            <material name="rover_wheels"/> </visual>
+    </link>
+    <joint name="camera_optical_joint" type="fixed">
+        <parent link="camera_link"/>
+        <child link="camera_link_optical"/>
+        <origin xyz="0 0 0" rpy="-1.5708 0 -1.5708"/>
+    </joint>
+    <link name="camera_link_optical"></link>
+    <joint name="lidar_joint" type="fixed">
+        <parent link="chassis"/>
+        <child link="lidar_link"/>
+        <origin xyz="-0.1 0 0.075" rpy="0 0 0"/>
+    </joint>
+    <link name="lidar_link">
+        <visual>
+            <geometry><cylinder radius="0.04" length="0.05"/></geometry>
+            <material name="rover_body"/>
+        </visual>
+    </link>
+    <joint name="imu_joint" type="fixed">
+        <parent link="chassis"/>
+        <child link="imu_link"/>
+        <origin xyz="0 0 0" rpy="0 0 0"/>
+    </joint>
+    <link name="imu_link"></link>
     <xacro:macro name="rover_wheel" params="prefix x_reflect y_reflect">
         <joint name="${prefix}_wheel_joint" type="continuous">
@@ -62,4 +122,14 @@
     <xacro:rover_wheel prefix="rear_left" x_reflect="-1" y_reflect="1"/>
     <xacro:rover_wheel prefix="rear_right" x_reflect="-1" y_reflect="-1"/>
+    <ros2_control name="RoverControl" type="system">
+        <hardware>
+            <plugin>ign_ros2_control/IgnitionSystem</plugin>
+        </hardware>
+        <joint name="camera_arm_joint">
+            <command_interface name="position"/>
+            <state_interface name="position"/>
+            <state_interface name="velocity"/>
+        </joint>
+    </ros2_control>
     <gazebo>
         <plugin filename="ignition-gazebo-diff-drive-system" name="ignition::gazebo::systems::DiffDrive">
@@ -78,3 +148,57 @@
         </plugin>
     </gazebo>
+    <gazebo reference="camera_link">
+        <sensor name="camera" type="camera">
+            <ignition_frame_id>camera_link_optical</ignition_frame_id>
+            <always_on>true</always_on>
+            <update_rate>30</update_rate>
+            <visualize>true</visualize>
+            <topic>camera/image_raw</topic>
+            <camera>
+                <horizontal_fov>1.089</horizontal_fov>
+                <image>
+                    <width>640</width>
+                    <height>480</height>
+                    <format>R8G8B8</format>
+                </image>
+                <clip><near>0.05</near><far>8.0</far></clip>
+            </camera>
+        </sensor>
+    </gazebo>
+    <gazebo reference="lidar_link">
+        <sensor name="lidar" type="gpu_lidar">
+            <ignition_frame_id>lidar_link</ignition_frame_id>
+            <always_on>true</always_on>
+            <update_rate>10</update_rate>
+            <visualize>true</visualize>
+            <topic>scan</topic>
+            <ray>
+                <scan>
+                    <horizontal>
+                        <samples>360</samples>
+                        <resolution>1.0</resolution>
+                        <min_angle>-3.14159</min_angle>
+                        <max_angle>3.14159</max_angle>
+                    </horizontal>
+                </scan>
+                <range>
+                    <min>0.12</min><max>3.5</max><resolution>0.015</resolution>
+                </range>
+            </ray>
+        </sensor>
+    </gazebo>
+    <gazebo reference="imu_link">
+        <sensor name="imu_sensor" type="imu">
+            <ignition_frame_id>imu_link</ignition_frame_id>
+            <always_on>true</always_on>
+            <update_rate>100</update_rate>
+            <visualize>true</visualize>
+            <topic>imu</topic>
+        </sensor>
+    </gazebo>
+    <gazebo>
+        <plugin filename="ign_ros2_control-system" name="ign_ros2_control::IgnitionROS2ControlPlugin">
+            <parameters>$(find rover_robot)/config/controllers.yaml</parameters>
+        </plugin>
+    </gazebo>
 </robot>

Commit message: updated

File: src/rover_robot/urdf/robot.urdf.xacro (robot description, xacro)
@@ -39,4 +39,5 @@
         <axis xyz="0 1 0"/>
         <limit lower="-0.785" upper="0.785" effort="10.0" velocity="1.0"/>
+        <dynamics damping="1.0" friction="0.5"/>
     </joint>
     <link name="camera_arm">
@@ -131,4 +132,24 @@
             <state_interface name="velocity"/>
         </joint>
+        <joint name="front_left_wheel_joint">
+            <command_interface name="velocity"/>
+            <state_interface name="position"/>
+            <state_interface name="velocity"/>
+        </joint>
+        <joint name="front_right_wheel_joint">
+            <command_interface name="velocity"/>
+            <state_interface name="position"/>
+            <state_interface name="velocity"/>
+        </joint>
+        <joint name="rear_left_wheel_joint">
+            <command_interface name="velocity"/>
+            <state_interface name="position"/>
+            <state_interface name="velocity"/>
+        </joint>
+        <joint name="rear_right_wheel_joint">
+            <command_interface name="velocity"/>
+            <state_interface name="position"/>
+            <state_interface name="velocity"/>
+        </joint>
     </ros2_control>
     <gazebo>

Commit message: updated

File: src/rover_robot/urdf/robot.urdf.xacro (robot description, xacro)
@@ -132,25 +132,14 @@
             <state_interface name="velocity"/>
         </joint>
-        <joint name="front_left_wheel_joint">
-            <command_interface name="velocity"/>
-            <state_interface name="position"/>
-            <state_interface name="velocity"/>
-        </joint>
-        <joint name="front_right_wheel_joint">
-            <command_interface name="velocity"/>
-            <state_interface name="position"/>
-            <state_interface name="velocity"/>
-        </joint>
-        <joint name="rear_left_wheel_joint">
-            <command_interface name="velocity"/>
-            <state_interface name="position"/>
-            <state_interface name="velocity"/>
-        </joint>
-        <joint name="rear_right_wheel_joint">
-            <command_interface name="velocity"/>
-            <state_interface name="position"/>
-            <state_interface name="velocity"/>
-        </joint>
     </ros2_control>
+    <gazebo>
+    <plugin filename="libignition-gazebo-joint-state-publisher-system.so" name="ignition::gazebo::systems::JointStatePublisher">
+        <topic>joint_states</topic>
+        <joint_name>front_left_wheel_joint</joint_name>
+        <joint_name>front_right_wheel_joint</joint_name>
+        <joint_name>rear_left_wheel_joint</joint_name>
+        <joint_name>rear_right_wheel_joint</joint_name>
+    </plugin>
+    </gazebo>
     <gazebo>
         <plugin filename="ignition-gazebo-diff-drive-system" name="ignition::gazebo::systems::DiffDrive">
@@ -162,5 +151,5 @@
             <wheel_radius>0.1</wheel_radius>
             <odom_publish_frequency>50</odom_publish_frequency>
-            <topic>cmd_vel</topic>
+            <topic>/cmd_vel</topic>
             <publish_odom>true</publish_odom>
             <publish_odom_tf>true</publish_odom_tf>
